File: Development/sphere_robo/sphere_robo.sch (EAGLE design)
At the start: 33 parts, among them IC1 ATMEGA328P-AU, J1 DM3AT-SF-PEJM5, U1 RN4020-V/RM123

Commit message: edit sphere_robo
Parts:
- added R16, R17: (no value), generic:RESISTOR1608_REDUCED
Changed lines of the file:
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@@
 <part name="C9" library="generic" deviceset="CAPACITOR-POL" device="PANASONIC_D"/>
 <part name="C10" library="generic" deviceset="CAPACITOR-POL" device="PANASONIC_D"/>
+<part name="R16" library="generic" deviceset="RESISTOR" device="1608_REDUCED"/>
+<part name="R17" library="generic" deviceset="RESISTOR" device="1608_REDUCED"/>
 </parts>
 <sheets>
@@
 <instance part="C9" gate="G$1" x="40.64" y="53.34"/>
 <instance part="C10" gate="G$1" x="50.8" y="53.34"/>
+<instance part="R16" gate="G$1" x="15.24" y="43.18"/>
+<instance part="R17" gate="G$1" x="25.4" y="43.18"/>
 </instances>
 <busses>

Commit message: sphere_robo 試作設計完了
Parts:
- added C11, C13, C14, C20: 1u, generic:CAPACITOR1608_REDUCED
- added C12: 2.2u, generic:CAPACITOR1608_REDUCED
- added C15: 0.01u, generic:CAPACITOR1608_REDUCED
- added C16, C23, C24: 10u, generic:CAPACITOR2012_REDUCED
- added C17, C18: 47u, generic:CAPACITOR-POLPANASONIC_F
- added C19, C21, C22, C27: 0.1u, generic:CAPACITOR1608_REDUCED
- added C25, C26: DNP, generic:CAPACITOR1608_REDUCED
- added IC2: LM4880, audio_amp:LM4880
- added IC3, IC4: BD6211F, motor_driver:BD6211F
- added LED4: (no value), generic:LED1608_REDUCED
- added M1, M2, PWR, SP2, SP3: M02NOSILK, header:M02NOSILK
- added R18, R21, R24: 10k, generic:RESISTOR1608_REDUCED
- added R19, R22: 20, generic:RESISTOR1608_REDUCED
- added R20, R23: 470, generic:RESISTOR1608_REDUCED
- added R25: 20k, generic:RESISTOR1608_REDUCED
- added R26, R34: (no value), generic:RESISTOR1608_REDUCED
- added R27: 100k, generic:RESISTOR1608_REDUCED
- added R28, R29, R30, R31: DNP, generic:RESISTOR1608_REDUCED
- added R32, R33: 0, generic:RESISTOR1608_REDUCED
- added SP1: UM1515A, speaker:UM1515A
- added SW1: 2MS1-T1-B4-VS2-Q-E, switch:2MS1-T1-B4-VS2-Q-E
- added U2: NJM2884U1, LDO:NJM2884U1
- added U3: UT7500G-18-AB3-B-R, LDO:UT7500G-18-AB3-B-R
- added X1: ABM2, crystal:ABM2
- C1, C2, C3, C4: value (none) -> 0.1u
- C10: value (none) -> 10u; device generic:CAPACITOR-POLPANASONIC_D -> generic:CAPACITOR2012_REDUCED
- C5: value (none) -> 1u
- C6: value (none) -> DNP
- C7, C8: value (none) -> 18p
- C9: value (none) -> 0.01u; device generic:CAPACITOR-POLPANASONIC_D -> generic:CAPACITOR1608_REDUCED
- R1, R13, R14, R15: value (none) -> 10k
- R11, R5: value 100k -> DNP
- R12: value 100k -> 1M
- R16, R17: value (none) -> 20k
- R2, R3, R4: value (none) -> 1k
Connections:
- removed net AGND: U$1.AGND0, U$1.AGND1, U$1.AGND2, U$1.AGND3
- new net FIN1: IC1.PC0(ADC0), IC3.FIN
- new net FIN2: IC1.PC2(ADC2), IC4.FIN
- new net INA: IC2.INA, R16.1, R17.2
- new net INB: IC2.INB, R25.2, R26.1
- new net LEFT: R19.1, R20.1, U$1.LEFT
- new net N$14: C18.-, SP1.+, SP3.2
- new net N$16: C9.2, R19.2
- new net N$18: R18.2, U2.CTL
- new net N$20: C10.1, R20.2
- new net N$21: C10.2, R17.1, R21.2
- new net N$23: C15.2, R22.2
- new net N$24: C16.1, R23.2
- new net N$25: C16.2, R24.2, R25.1
- new net N$26: C20.2, IC2.BYPASS
- new net N$29: C17.-, SP2.2
- new net N$31: LED4.A, R34.1
- new net N$35: C25.2, IC3.VREF, R28.2, R31.1, R32.2
- new net N$36: C26.2, IC4.VREF, R29.2, R30.1, R33.2
- new net N$37: IC4.OUT1, M2.2
- new net N$38: IC4.OUT2, M2.1
- new net N$39: IC3.OUT1, M1.2
- new net N$40: IC3.OUT2, M1.1
- new net OUTA: C17.+, IC2.OUTA, R16.2
- new net OUTB: C18.+, IC2.OUTB, R26.2
- new net RIGHT: R22.1, R23.1, U$1.RIGHT
- new net RIN1: IC1.PC1(ADC1), IC3.RIN
- new net RIN2: IC1.PC3(ADC3), IC4.RIN
- new net SHUTDOWN: IC1.PB2(SS/OC1B), IC2.SHUTDOWN, R27.1
- new net VCC: C11.2, C19.1, C21.1, C22.1, C23.1, C24.1, IC2.VDD, IC3.VCC@1, IC3.VCC@2, IC4.VCC@1, IC4.VCC@2, R18.1, SW1.1, U2.VIN
- new net VREF1: IC1.PD3(INT1), R32.1
- new net VREF2: IC1.PD5(T1), R33.1
- net +1V8: now also C14.2, U3.VOUT
- net +3V3: now also C12.2, C13.2, C27.1, R28.1, R29.1, R34.2, U2.VOUT, U3.VIN
- net CMD/MLDP: now also IC1.PD4(XCK/T0); no longer IC1.PC2(ADC2)
- net GND: now also C11.1, C12.1, C13.1, C14.1, C15.1, C19.2, C20.1, C21.2, C22.2, C23.2, C24.2, C25.1, C26.1, C27.2, C9.1, IC2.GND, IC3.GND, IC4.GND, LED4.K, PWR.1, R21.1, R24.1, R27.2, R30.2, R31.2, SP1.-, SP2.1, SP3.1, U$1.AGND0, U$1.AGND1, U$1.AGND2, U$1.AGND3, U2.GND, U3.GND
- net N$13: now also PWR.2, SW1.2; no longer U$1.LEFT
- net N$15: now also X1.P$2
- net N$19: now also X1.P$1
- net WAKE_HW: now also IC1.ADC6; no longer IC1.PC1(ADC1)
- net WAKE_SW: now also IC1.ADC7; no longer IC1.PC0(ADC0)
Other:
- moved on the sheet: C2, R16, R17
