File: Development/sphere_robo/sphere_robo.sch (EAGLE design)
At the start: 34 parts, among them IC1 ATMEGA328P-AU, IC3 BD6211F, IC4 BD6211F, M1 M02NOSILK, M2 M02NOSILK, SW2 SK-12D01-VG4, U1 RN4020-V/RM123, U2 NJM2884U1

Commit message: rev3設計完了
Parts:
- removed C21: 0.1u, generic:CAPACITOR1608_REDUCED
- removed C23: 10u, generic:CAPACITOR2012_REDUCED
- removed LED2, LED3: (no value), generic:LED1608_REDUCED
- removed R15, R18: 10k, generic:RESISTOR1608_REDUCED
- removed R27: 100k, generic:RESISTOR1608_REDUCED
- removed R34: (no value), generic:RESISTOR1608_REDUCED
- added C10, C5, C8, C9: 0.1u, generic:CAPACITOR1608_REDUCED
- added IC2: BD6211F, motor_driver:BD6211F
- added J1: M03X2STD, header:M03X2STD
- added JP2: M02NOSILK, header:M02NOSILK
- added JP3, JP4: (no value), header:M06NOSILK
- added R6: 10k, generic:RESISTOR1608_REDUCED
- added R8: 1k, generic:RESISTOR1608_REDUCED
- C1: value 0.1u -> 1u
- C11: value 1u -> 10u; device generic:CAPACITOR1608_REDUCED -> generic:CAPACITOR2012_REDUCED
- C12: value 2.2u -> 10u; device generic:CAPACITOR1608_REDUCED -> generic:CAPACITOR2012_REDUCED
- C2: value 0.1u -> 2.2u
- C3: value 0.1u -> 10u; device generic:CAPACITOR1608_REDUCED -> generic:CAPACITOR2012_REDUCED
- IC1: value ATMEGA328P-AU -> BD6211F; device AVR:ATMEGA328P-AU -> motor_driver:BD6211F
- IC3: value BD6211F -> ATMEGA328P-AU; device motor_driver:BD6211F -> AVR:ATMEGA328P-AU
- IC4: value BD6211F -> XCL101; device motor_driver:BD6211F -> DCDC:XCL101
- JP1: value (none) -> M02NOSILK; device header:M06NOSILK -> header:M02NOSILK
- R2: value 1k -> (none)
- R3, R4: value 1k -> 10k
- U1: value RN4020-V/RM123 -> NJM2884U1; device com_module:RN4020-V/RM123 -> LDO:NJM2884U1
- U2: value NJM2884U1 -> RN4020-V/RM123; device LDO:NJM2884U1 -> com_module:RN4020-V/RM123
- renumbered C22 to C7, C24 to C6, LED1 to CONNECTION, LED4 to POWER, R13 to R7, R14 to R5, SW2 to SW1
Connections:
- removed net N$1: C3.2, IC1.PC6(/RESET), R1.2
- removed net N$4: LED2.A, R3.2
- removed net N$5: LED3.A, R4.2
- removed net PIO2: R3.1, U1.MLDP_EV/PIO2/CS
- removed net PIO3: R4.1, U1.WS/PIO3/MOSI
- removed net SHUTDOWN: IC1.PB2(SS/OC1B), R27.1
- new net N$20: IC4.L1, IC4.LX
- new net N$7: IC3.PC5(ADC5/SCL), R6.1
- new net RST: C5.2, IC3.PC6(/RESET), J1.5, R3.2
- net +3V3: now also C10.1, C12.1, C8.2, C9.2, IC3.AREF, IC3.AVCC, IC3.VCC@1, IC3.VCC@2, IC4.VOUT, J1.2, JP1.1, JP3.3, JP4.3, R2.2, R3.1, R4.1, U1.VOUT, U2.VDD; no longer C1.1, C12.2, C4.2, IC1.AREF, IC1.AVCC, IC1.VCC@1, IC1.VCC@2, JP1.3, R1.1, R15.1, R34.2, U1.VDD, U2.VOUT
- net BLE_RX: now also JP4.4, R6.2, U2.UART_RX; no longer IC1.PC5(ADC5/SCL), U1.UART_RX
- net BLE_TX: now also IC3.PC4(ADC4/SDA), JP4.5, U2.UART_TX; no longer IC1.PC4(ADC4/SDA), U1.UART_TX
- net CMD/MLDP: now also IC3.PD6(AIN0), U2.CMD/MLDP; no longer U1.CMD/MLDP
- net FIN1: now also IC1.FIN, IC3.PC0(ADC0); no longer IC1.PC0(ADC0), IC3.FIN
- net FIN2: now also IC2.FIN, IC3.PC2(ADC2); no longer IC1.PC2(ADC2), IC4.FIN
- net GND: now also C1.1, C10.2, C11.2, C12.2, C3.2, C4.2, C8.1, C9.1, IC2.GND, IC3.GND@1, IC3.GND@2, IC4.VSS, J1.6, JP1.2, JP2.2, JP3.1, JP4.1, U1.GND, U2.GND@1, U2.GND@2, U2.GND@3, U2.GND@4; no longer C1.2, C11.1, C12.1, C21.2, C23.2, C4.1, IC1.GND@1, IC1.GND@2, IC4.GND, JP1.1, LED2.K, LED3.K, R27.2, U1.GND@1, U1.GND@2, U1.GND@3, U1.GND@4, U2.GND
- net MISO: now also IC3.PB4(MISO), J1.1; no longer IC1.PB4(MISO)
- net MOSI: now also IC3.PB3(MOSI/OC2), J1.4; no longer IC1.PB3(MOSI/OC2)
- net N$11: now also U2.SPI/!PIO; no longer U1.SPI/!PIO
- net N$18: now also R1.2, U1.CTL; no longer R18.2, U2.CTL
- net N$2: now also C5.1, JP3.6; no longer C3.1, JP1.6
- net N$3: now also R8.2; no longer R2.2
- net N$31: now also R2.1; no longer R34.1
- net N$37: now also IC2.OUT1; no longer IC4.OUT1
- net N$38: now also IC2.OUT2; no longer IC4.OUT2
- net N$39: now also IC1.OUT1; no longer IC3.OUT1
- net N$40: now also IC1.OUT2; no longer IC3.OUT2
- net PIO1: now also R8.1, U2.PIO1/SCK; no longer R2.1, U1.PIO1/SCK
- net RIN1: now also IC1.RIN, IC3.PC1(ADC1); no longer IC1.PC1(ADC1), IC3.RIN
- net RIN2: now also IC2.RIN, IC3.PC3(ADC3); no longer IC1.PC3(ADC3), IC4.RIN
- net RXD: now also IC3.PD0(RXD), JP3.4; no longer IC1.PD0(RXD), JP1.4
- net SCK: now also IC3.PB5(SCK), J1.3; no longer IC1.PB5(SCK)
- net TXD: now also IC3.PD1(TXD), JP3.5; no longer IC1.PD1(TXD), JP1.5
- net VCC: now also C1.2, C11.1, C3.1, C4.1, IC1.VCC@1, IC1.VCC@2, IC2.VCC@1, IC2.VCC@2, IC4.CE, IC4.L2, IC4.VBAT, JP2.1, R1.1, U1.VIN; no longer C11.2, C21.1, C23.1, IC3.VCC@1, IC3.VCC@2, IC4.VCC@1, IC4.VCC@2, R18.1, U2.VIN
- net VREF1: now also IC1.VREF, IC3.PD3(INT1); no longer IC1.PD3(INT1), IC3.VREF
- net VREF2: now also IC2.VREF, IC3.PD5(T1); no longer IC1.PD5(T1), IC4.VREF
- net WAKE_HW: now also R4.2, U2.WAKE_HW; no longer IC1.ADC6, R15.2, U1.WAKE_HW
- net WAKE_SW: now also U2.WAKE_SW; no longer IC1.ADC7, U1.WAKE_SW
Other:
- moved on the sheet: C1, C11, C12, C2, C3, C4, IC4, R1, R2, R3, R4

Commit message: 抵抗値変更
Parts:
- R6: value 10k -> 100
Changed lines of the file:
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@@
 <part name="J1" library="header" deviceset="M03X2" device="STD"/>
 <part name="+3V311" library="supply" deviceset="+3V3" device=""/>
-<part name="R6" library="generic" deviceset="RESISTOR" device="1608_REDUCED" value="10k"/>
+<part name="R6" library="generic" deviceset="RESISTOR" device="1608_REDUCED" value="100"/>
 <part name="JP4" library="header" deviceset="M06" device="NOSILK"/>
 <part name="GND14" library="supply" deviceset="GND" device=""/>
