File: Development/sphere_robo/sphere_robo.brd (EAGLE design)
At the start: 100 x 80 mm, 33 parts, among them IC1 ATMEGA328P-AU, J1 DM3AT-SF-PEJM5, U1 RN4020-V/RM123

Commit message: edit sphere_robo
Parts:
- added R16, R17: (no value), generic:SMD1608_REDUCED
Changed lines of the file:
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@@
 <element name="C9" library="generic" package="PANASONIC_D" value="" x="-38" y="-143"/>
 <element name="C10" library="generic" package="PANASONIC_D" value="" x="-38" y="-150"/>
+<element name="R16" library="generic" package="SMD1608_REDUCED" value="" x="-45" y="-156"/>
+<element name="R17" library="generic" package="SMD1608_REDUCED" value="" x="-45" y="-159"/>
 </elements>
 <signals>

Commit message: sphere_robo 試作設計完了
Parts:
- added C11, C13, C14, C20: 1u, generic:SMD1608_REDUCED
- added C12: 2.2u, generic:SMD1608_REDUCED
- added C15: 0.01u, generic:SMD1608_REDUCED
- added C16, C23, C24: 10u, generic:SMD2012_REDUCED
- added C17, C18: 47u, generic:PANASONIC_F
- added C19, C21, C22, C27: 0.1u, generic:SMD1608_REDUCED
- added C25, C26, R28, R29, R30, R31: DNP, generic:SMD1608_REDUCED
- added IC2: LM4880, audio_amp:SOIC-8
- added IC3, IC4: BD6211F, motor_driver:SOP-8
- added LED4: (no value), generic:LED1608_REDUCED
- added M1, M2, PWR, SP2, SP3: M02NOSILK, header:1X02-NOSILK
- added R18, R21, R24: 10k, generic:SMD1608_REDUCED
- added R19, R22: 20, generic:SMD1608_REDUCED
- added R20, R23: 470, generic:SMD1608_REDUCED
- added R25: 20k, generic:SMD1608_REDUCED
- added R26, R34: (no value), generic:SMD1608_REDUCED
- added R27: 100k, generic:SMD1608_REDUCED
- added R32, R33: 0, generic:SMD1608_REDUCED
- added SP1: UM1515A, speaker:UM1515IA085008LFMP
- added SW1: 2MS1-T1-B4-VS2-Q-E, switch:2MS1-T1-B4-VS2-Q-E
- added U2: NJM2884U1, LDO:SOT-89-5
- added U3: UT7500G-18-AB3-B-R, LDO:SOT-89
- added X1: ABM2, crystal:ABM2
- C1, C2, C3, C4: value (none) -> 0.1u
- C10: value (none) -> 10u; device generic:PANASONIC_D -> generic:SMD2012_REDUCED
- C5: value (none) -> 1u
- C6: value (none) -> DNP
- C7, C8: value (none) -> 18p
- C9: value (none) -> 0.01u; device generic:PANASONIC_D -> generic:SMD1608_REDUCED
- R1, R13, R14, R15: value (none) -> 10k
- R11, R5: value 100k -> DNP
- R12: value 100k -> 1M
- R16, R17: value (none) -> 20k
- R2, R3, R4: value (none) -> 1k
- moved R16 225.0 mm to (39.3, 52.6), turned to 90 degrees
- moved R17 224.9 mm to (39.3, 49.5), turned to 90 degrees
- moved C10 202.9 mm to (35.5, 39.1)
- moved C9 192.8 mm to (29.0, 37.8), turned to 180 degrees
- moved C8 171.1 mm to (3.90, 37.1), turned to 270 degrees
- moved R14 165.0 mm to (23.1, 15.9)
- moved C6 164.6 mm to (24.3, 35.2), turned to 90 degrees
- moved C7 164.5 mm to (3.89, 34.0), turned to 90 degrees
- moved R12 160.8 mm to (2.71, 35.6), turned to 90 degrees
- moved R11 158.5 mm to (22.0, 34.7)
- moved R15 158.0 mm to (19.3, 6.10)
- moved R10 157.9 mm to (16.2, 41.7), turned to 90 degrees
- moved C5 151.7 mm to (22.0, 36.0)
- moved R13 149.7 mm to (19.2, 4.71), turned to 180 degrees
- moved R9 139.1 mm to (19.9, 28.1)
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Connections:
- removed net AGND: U$1.P$37, U$1.P$40, U$1.P$41, U$1.P$47
- new net FIN1: IC1.23, IC3.4
- new net FIN2: IC1.25, IC4.4
- new net INA: IC2.2, R16.1, R17.2
- new net INB: IC2.6, R25.2, R26.1
- new net LEFT: R19.1, R20.1, U$1.P$46
- new net N$14: C18.-, SP1.1, SP3.2
- new net N$16: C9.2, R19.2
- new net N$18: R18.2, U2.1
- new net N$20: C10.1, R20.2
- new net N$21: C10.2, R17.1, R21.2
- new net N$23: C15.2, R22.2
- new net N$24: C16.1, R23.2
- new net N$25: C16.2, R24.2, R25.1
- new net N$26: C20.2, IC2.3
- new net N$29: C17.-, SP2.2
- new net N$31: LED4.A, R34.1
- new net N$35: C25.2, IC3.6, R28.2, R31.1, R32.2
- new net N$36: C26.2, IC4.6, R29.2, R30.1, R33.2
- new net N$37: IC4.1, M2.2
- new net N$38: IC4.7, M2.1
- new net N$39: IC3.1, M1.2
- new net N$40: IC3.7, M1.1
- new net OUTA: C17.+, IC2.1, R16.2
- new net OUTB: C18.+, IC2.7, R26.2
- new net RIGHT: R22.1, R23.1, U$1.P$39
- new net RIN1: IC1.24, IC3.5
- new net RIN2: IC1.26, IC4.5
- new net SHUTDOWN: IC1.14, IC2.5, R27.1
- new net VCC: C11.2, C19.1, C21.1, C22.1, C23.1, C24.1, IC2.8, IC3.2, IC3.3, IC4.2, IC4.3, R18.1, SW1.1, U2.5
- new net VREF1: IC1.1, R32.1
- new net VREF2: IC1.9, R33.1
- net +1V8: now also C14.2, U3.1
- net +3V3: now also C12.2, C13.2, C27.1, R28.1, R29.1, R34.2, U2.4, U3.3
- net CMD/MLDP: now also IC1.2; no longer IC1.25
- net GND: now also C11.1, C12.1, C13.1, C14.1, C15.1, C19.2, C20.1, C21.2, C22.2, C23.2, C24.2, C25.1, C26.1, C27.2, C9.1, IC2.4, IC3.8, IC4.8, LED4.K, PWR.1, R21.1, R24.1, R27.2, R30.2, R31.2, SP1.2, SP2.1, SP3.1, U$1.P$37, U$1.P$40, U$1.P$41, U$1.P$47, U2.2, U3.2, U3.4
- net N$13: now also PWR.2, SW1.2; no longer U$1.P$46
- net N$15: now also X1.2
- net N$19: now also X1.1
- net WAKE_HW: now also IC1.19; no longer IC1.24
- net WAKE_SW: now also IC1.22; no longer IC1.23
Routing:
- net GND: track 0.00 -> 416.5 mm, vias 0 -> 104
- net +3V3: track 0.00 -> 180.8 mm, vias 0 -> 10
- net VCC: track 0.00 -> 86.1 mm
- net VREF1: track 0.00 -> 68.6 mm, vias 0 -> 2
- net SHUTDOWN: track 0.00 -> 59.7 mm, vias 0 -> 2
- net SCK: track 0.00 -> 51.3 mm, vias 0 -> 3
- net MISO: track 0.00 -> 51.2 mm, vias 0 -> 3
- net MOSI: track 0.00 -> 49.4 mm, vias 0 -> 3
- net SD-CS: track 0.00 -> 41.3 mm, vias 0 -> 2
- net +1V8: track 0.00 -> 38.6 mm, vias 0 -> 2
- net BLE_RX: track 0.00 -> 32.4 mm, vias 0 -> 2
- net BLE_TX: track 0.00 -> 31.9 mm, vias 0 -> 2
- net CMD/MLDP: track 0.00 -> 31.3 mm, vias 0 -> 2
- net WAKE_SW: track 0.00 -> 31.1 mm, vias 0 -> 2
- net WAKE_HW: track 0.00 -> 29.6 mm, vias 0 -> 2
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- added copper zone on layer 1, net GND
- added copper zone on layer 16, net GND
Other:
- board size 100 x 80 mm -> 60 x 60 mm
- board text added: "+"
- board text added: "-"
- board text added: "3V3"
- board text added: "GND"
- board text added: "KENBISHI"
- board text added: "M1"
- board text added: "M2"
- board text added: "Rev1"
- board text added: "SP2"
- board text added: "SP3"
- board text added: "SPHERE_ROBO"
