File: Development/sphere_robo/sphere_robo.brd (EAGLE design)
At the start: 60 x 60 mm, 34 parts, among them IC1 ATMEGA328P-AU, IC3 BD6211F, IC4 BD6211F, M1 M02NOSILK, M2 M02NOSILK, SW2 SK-12D01-VG4, U1 RN4020-V/RM123, U2 NJM2884U1

Commit message: rev3設計完了
Parts:
- removed C21, C22: 0.1u, generic:SMD1608_REDUCED
- removed C23, C24: 10u, generic:SMD2012_REDUCED
- removed LED1, LED2, LED3, LED4: (no value), generic:LED1608_REDUCED
- removed R13, R14, R15, R18: 10k, generic:SMD1608_REDUCED
- removed R27: 100k, generic:SMD1608_REDUCED
- removed R34: (no value), generic:SMD1608_REDUCED
- removed SW2: SK-12D01-VG4, switch:SK-12D01-VG4
- added C10, C5, C7, C8, C9: 0.1u, generic:SMD1608_REDUCED
- added C6: 10u, generic:SMD2012_REDUCED
- added CONNECTION, POWER: (no value), generic:LED1608_REDUCED
- added IC2: BD6211F, motor_driver:SOP-8
- added J1: M03X2STD, header:2X03
- added JP2: M02NOSILK, header:1X02-NOSILK
- added JP3, JP4: (no value), header:1X06-NOSILK
- added R5, R6, R7: 10k, generic:SMD1608_REDUCED
- added R8: 1k, generic:SMD1608_REDUCED
- added SW1: SK-12D01-VG4, switch:SK-12D01-VG4
- C1: value 0.1u -> 1u
- C11: value 1u -> 10u; device generic:SMD1608_REDUCED -> generic:SMD2012_REDUCED
- C12: value 2.2u -> 10u; device generic:SMD1608_REDUCED -> generic:SMD2012_REDUCED
- C2: value 0.1u -> 2.2u
- C3: value 0.1u -> 10u; device generic:SMD1608_REDUCED -> generic:SMD2012_REDUCED
- IC1: value ATMEGA328P-AU -> BD6211F; device AVR:TQFP32-08 -> motor_driver:SOP-8
- IC3: value BD6211F -> ATMEGA328P-AU; device motor_driver:SOP-8 -> AVR:TQFP32-08
- IC4: value BD6211F -> XCL101; device motor_driver:SOP-8 -> DCDC:CL-2025
- JP1: value (none) -> M02NOSILK; device header:1X06-NOSILK -> header:1X02-NOSILK
- R2: value 1k -> (none)
- R3, R4: value 1k -> 10k
- U1: value RN4020-V/RM123 -> NJM2884U1; device com_module:RN4020 -> LDO:SOT-89-5
- U2: value NJM2884U1 -> RN4020-V/RM123; device LDO:SOT-89-5 -> com_module:RN4020
- moved C2 47.0 mm to (17.3, 41.1)
- moved R2 33.1 mm to (9.80, 42.5), turned to 0 degrees
- moved U2 33.1 mm to (22.2, 14.5)
- moved IC1 32.2 mm to (41.0, 37.0)
- moved U1 30.8 mm to (16.4, 44.2)
- moved C3 29.0 mm to (35.5, 38.0), turned to 180 degrees
- moved C1 28.4 mm to (20.2, 45.0)
- moved R3 25.1 mm to (13.9, 33.9), turned to 270 degrees
- moved IC4 24.6 mm to (22.0, 39.3)
- moved C4 22.9 mm to (35.5, 35.5), turned to 180 degrees
- moved JP1 22.7 mm to (12.2, 38.0), turned to 180 degrees
- moved M2 22.1 mm to (51.0, 47.5), turned to 180 degrees
- moved R1 21.3 mm to (19.4, 47.3), turned to 180 degrees
- moved M1 20.7 mm to (44.5, 47.5), turned to 180 degrees
- moved IC3 19.2 mm to (14.5, 26.5)
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Connections:
- removed net N$1: C3.2, IC1.29, R1.2
- removed net N$4: LED2.A, R3.2
- removed net N$5: LED3.A, R4.2
- removed net PIO2: R3.1, U1.11
- removed net PIO3: R4.1, U1.12
- removed net SHUTDOWN: IC1.14, R27.1
- new net N$20: IC4.1, IC4.7
- new net N$7: IC3.28, R6.1
- new net RST: C5.2, IC3.29, J1.5, R3.2
- net +3V3: now also C10.1, C12.1, C8.2, C9.2, IC3.18, IC3.20, IC3.4, IC3.6, IC4.2, J1.2, JP1.1, JP3.3, JP4.3, R2.2, R3.1, R4.1, R5.1, U1.4, U2.23; no longer C1.1, C12.2, C4.2, IC1.18, IC1.20, IC1.4, IC1.6, JP1.3, R1.1, R14.1, R15.1, R34.2, U1.23, U2.4
- net BLE_RX: now also JP4.4, R6.2, U2.6; no longer IC1.28, U1.6
- net BLE_TX: now also IC3.27, JP4.5, U2.5; no longer IC1.27, U1.5
- net CMD/MLDP: now also IC3.10, U2.8; no longer U1.8
- net FIN1: now also IC1.4, IC3.23; no longer IC1.23, IC3.4
- net FIN2: now also IC2.4, IC3.25; no longer IC1.25, IC4.4
- net GND: now also C1.1, C10.2, C11.2, C12.2, C3.2, C4.2, C6.2, C7.2, C8.1, C9.1, CONNECTION.K, IC1.8, IC2.8, IC3.21, IC3.3, IC3.5, IC4.6, J1.6, JP1.2, JP2.2, JP3.1, JP4.1, POWER.K, R7.2, U1.2, U2.1, U2.16, U2.24, U2.9; no longer C1.2, C11.1, C12.1, C21.2, C22.2, C23.2, C24.2, C4.1, IC1.21, IC1.3, IC1.5, IC3.8, IC4.8, JP1.1, LED1.K, LED2.K, LED3.K, LED4.K, R13.2, R27.2, U1.1, U1.16, U1.24, U1.9, U2.2
- net MISO: now also IC3.16, J1.1; no longer IC1.16
- net MOSI: now also IC3.15, J1.4; no longer IC1.15
- net N$11: now also R7.1, U2.17; no longer R13.1, U1.17
- net N$13: now also SW1.2; no longer SW2.2
- net N$18: now also R1.2, U1.1; no longer R18.2, U2.1
- net N$2: now also C5.1, JP3.6; no longer C3.1, JP1.6
- net N$3: now also CONNECTION.A, R8.2; no longer LED1.A, R2.2
- net N$31: now also POWER.A, R2.1; no longer LED4.A, R34.1
- net N$37: now also IC2.1; no longer IC4.1
- net N$38: now also IC2.7; no longer IC4.7
- net N$39: now also IC1.1; no longer IC3.1
- net N$40: now also IC1.7; no longer IC3.7
- net PIO1: now also R8.1, U2.10; no longer R2.1, U1.10
- net RIN1: now also IC1.5, IC3.24; no longer IC1.24, IC3.5
- net RIN2: now also IC2.5, IC3.26; no longer IC1.26, IC4.5
- net RXD: now also IC3.30, JP3.4; no longer IC1.30, JP1.4
- net SCK: now also IC3.17, J1.3; no longer IC1.17
- net TXD: now also IC3.31, JP3.5; no longer IC1.31, JP1.5
- net VCC: now also C1.2, C11.1, C3.1, C4.1, C6.1, C7.1, IC1.2, IC1.3, IC2.2, IC2.3, IC4.4, IC4.8, JP2.1, R1.1, SW1.1, U1.5; no longer C11.2, C21.1, C22.1, C23.1, C24.1, IC3.2, IC3.3, IC4.2, R18.1, SW2.1, U2.5
- net VREF1: now also IC1.6, IC3.1; no longer IC1.1, IC3.6
- net VREF2: now also IC2.6, IC3.9; no longer IC1.9, IC4.6
- net WAKE_HW: now also R4.2, U2.15; no longer IC1.19, R15.2, U1.15
- net WAKE_SW: now also R5.2, U2.7; no longer IC1.22, R14.2, U1.7
Routing:
- net GND: track 190.1 -> 60.4 mm, vias 89 -> 93
- net SHUTDOWN: track 59.0 -> 0.00 mm, vias 2 -> 0
- net MOSI: track 46.2 -> 5.36 mm, vias 3 -> 0
- net SCK: track 47.0 -> 11.6 mm, vias 3 -> 0
- net RST: track 0.00 -> 35.1 mm
- net MISO: track 49.0 -> 16.3 mm, vias 3 -> 0
- net VREF1: track 85.9 -> 54.8 mm, vias 4 -> 2
- net +3V3: track 141.7 -> 170.6 mm, vias 10 -> 1
- net WAKE_SW: track 31.1 -> 3.31 mm, vias 2 -> 0
- net FIN2: track 19.3 -> 46.9 mm, vias 0 -> 2
- net VCC: track 79.9 -> 104.2 mm
- net RIN2: track 26.5 -> 47.6 mm, vias 0 -> 2
- net N$7: track 0.00 -> 19.7 mm, vias 0 -> 2
- net VREF2: track 39.4 -> 57.1 mm, vias 4 -> 2
- net FIN1: track 23.7 -> 40.7 mm
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Other:
- outline, holes or cut-outs redrawn
- board text added: "Rev2"
- board text removed: "Rev1"
- board text removed: "SP2"
- board text removed: "SP3"

Commit message: 抵抗値変更
Parts:
- R6: value 10k -> 100
Changed lines of the file:
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@@
 <element name="SW1" library="switch" package="SK-12D01-VG4" value="SK-12D01-VG4" x="30" y="53.5" rot="R180"/>
 <element name="J1" library="header" package="2X03" value="M03X2STD" x="13.8" y="16.7" rot="R90"/>
-<element name="R6" library="generic" package="SMD1608_REDUCED" value="10k" x="27.1" y="19.9" rot="R270"/>
+<element name="R6" library="generic" package="SMD1608_REDUCED" value="100" x="27.1" y="19.9" rot="R270"/>
 <element name="JP4" library="header" package="1X06-NOSILK" value="" x="39.2" y="24.2" rot="R180"/>
 <element name="JP1" library="header" package="1X02-NOSILK" value="M02NOSILK" x="12.2" y="38" rot="R180"/>
