File: Development/hemisphere_robo/hemisphere_robo.brd (EAGLE design)
At the start: 100 x 50 mm, 74 parts, among them IC1 VS1053B, IC2 ATMEGA328P-AU, IC3 HT82V739, IC4 BD6211F, IC5 BD6211F, IC6 BD6211F, J1 M03X2STD, J2 DM3AT-SF-PEJM5, U1 NJM2884U1, U2 UT7500G-18-AB3-B-R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

Commit message: 抵抗値変更
Parts:
- R16, R17, R18: value 10k -> 47
Changed lines of the file:
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@@
 <attribute name="VALUE" x="10.15" y="42.2" size="0.8128" layer="27" font="vector" rot="R90"/>
 </element>
-<element name="R16" library="generic" package="SMD1608_REDUCED" value="10k" x="8.5" y="39.9" smashed="yes" rot="R90">
+<element name="R16" library="generic" package="SMD1608_REDUCED" value="47" x="8.5" y="39.9" smashed="yes" rot="R90">
 <attribute name="NAME" x="7.85" y="39.1" size="0.8128" layer="25" font="vector" rot="R90"/>
 <attribute name="VALUE" x="10.15" y="39.1" size="0.8128" layer="27" font="vector" rot="R90"/>
 </element>
-<element name="R17" library="generic" package="SMD1608_REDUCED" value="10k" x="8.5" y="30.2" smashed="yes" rot="R90">
+<element name="R17" library="generic" package="SMD1608_REDUCED" value="47" x="8.5" y="30.2" smashed="yes" rot="R90">
 <attribute name="NAME" x="7.85" y="29.4" size="0.8128" layer="25" font="vector" rot="R90"/>
 <attribute name="VALUE" x="10.15" y="29.4" size="0.8128" layer="27" font="vector" rot="R90"/>
@@
 <attribute name="VALUE" x="10.15" y="32.5" size="0.8128" layer="27" font="vector" rot="R90"/>
 </element>
-<element name="R18" library="generic" package="SMD1608_REDUCED" value="10k" x="8.5" y="20.4" smashed="yes" rot="R90">
+<element name="R18" library="generic" package="SMD1608_REDUCED" value="47" x="8.5" y="20.4" smashed="yes" rot="R90">
 <attribute name="NAME" x="7.85" y="19.6" size="0.8128" layer="25" font="vector" rot="R90"/>
 <attribute name="VALUE" x="10.15" y="19.6" size="0.8128" layer="27" font="vector" rot="R90"/>
