File: Development/hemisphere_robo/hemisphere_robo.sch (EAGLE design)
At the start: 83 parts, among them IC1 ATMEGA328P-AU, IC2 LM4880, IC3 BD6211F, IC4 BD6211F, J1 DM3AT-SF-PEJM5, M1 M02NOSILK, M2 M02NOSILK, SW1 2MS1-T1-B4-VS2-Q-E, U1 RN4020-V/RM123, U2 NJM2884U1, U3 UT7500G-18-AB3-B-R, X1 ABM2

Commit message: 設計完了
Parts:
- removed LED4: (no value), generic:LED1608_REDUCED
- removed M1, M2, PWR, SP3: M02NOSILK, header:M02NOSILK
- removed R19, R22: 20, generic:RESISTOR1608_REDUCED
- removed R20, R23: 470, generic:RESISTOR1608_REDUCED
- removed R21, R24: 10k, generic:RESISTOR1608_REDUCED
- removed R25: 20k, generic:RESISTOR1608_REDUCED
- removed R26, R34: (no value), generic:RESISTOR1608_REDUCED
- removed R27: 100k, generic:RESISTOR1608_REDUCED
- removed R28, R29, R30, R31: DNP, generic:RESISTOR1608_REDUCED
- removed R32, R33: 0, generic:RESISTOR1608_REDUCED
- removed SP1: UM1515A, speaker:UM1515A
- removed SW1: 2MS1-T1-B4-VS2-Q-E, switch:2MS1-T1-B4-VS2-Q-E
- removed U$1: VS1053B, MP3:VS1053B
- added BAT1: BH-331-3P24, battery:BH-331-3P24
- added C28, C29, C30: 0.1u, generic:CAPACITOR1608_REDUCED
- added IC5, IC6: BD6211F, motor_driver:BD6211F
- added J2: DM3AT-SF-PEJM5, SDcard:DM3AT-SF-PEJM5
- added JP2, JP7, JP8, JP9: M02NOSILK, header:M02NOSILK
- added JP3, JP4: (no value), header:M06NOSILK
- added JP5: (no value), header:M03NOSILK
- added VR1: VR, VR:VR
- C1: value 0.1u -> 1u
- C10, C16: value 10u -> 1u; device generic:CAPACITOR2012_REDUCED -> generic:CAPACITOR1608_REDUCED
- C12: value 2.2u -> DNP
- C13, C5: value 1u -> 0.1u
- C14: value 1u -> 0.01u
- C15: value 0.01u -> 10u; device generic:CAPACITOR1608_REDUCED -> generic:CAPACITOR2012_REDUCED
- C17: value 47u -> 1u; device generic:CAPACITOR-POLPANASONIC_F -> generic:CAPACITOR1608_REDUCED
- C18: value 47u -> 0.1u; device generic:CAPACITOR-POLPANASONIC_F -> generic:CAPACITOR1608_REDUCED
- C2, C3: value 0.1u -> 18p
- C20: value 1u -> (none); device generic:CAPACITOR1608_REDUCED -> generic:CAPACITOR-POLPANASONIC_D
- C21: value 0.1u -> (none); device generic:CAPACITOR1608_REDUCED -> generic:CAPACITOR-POLPANASONIC_D
- C22: value 0.1u -> 10u; device generic:CAPACITOR1608_REDUCED -> generic:CAPACITOR2012_REDUCED
- C25, C26, C6: value DNP -> 0.1u
- C7: value 18p -> 2.2u
- C8: value 18p -> 0.1u
- C9: value 0.01u -> 1u
- IC1: value ATMEGA328P-AU -> VS1053B; device AVR:ATMEGA328P-AU -> MP3:VS1053B
- IC2: value LM4880 -> ATMEGA328P-AU; device audio_amp:LM4880 -> AVR:ATMEGA328P-AU
- IC3: value BD6211F -> HT82V739; device motor_driver:BD6211F -> audio_amp:HT82V739
- J1: value DM3AT-SF-PEJM5 -> M03X2STD; device SDcard:DM3AT-SF-PEJM5 -> header:M03X2STD
- JP1: value (none) -> M02NOSILK; device header:M06NOSILK -> header:M02NOSILK
- R11: value DNP -> 20
- R12: value 1M -> 10k
- R14: value 10k -> 1k
- R16, R17: value 20k -> 10k
- R2: value 1k -> 1M
- R3: value 1k -> 10k
- R4: value 1k -> (none)
- R7: value 100k -> 1k
- R8: value 100k -> 470
- R9: value 100k -> DNP
- U1: value RN4020-V/RM123 -> NJM2884U1; device com_module:RN4020-V/RM123 -> LDO:NJM2884U1
- U2: value NJM2884U1 -> UT7500G-18-AB3-B-R; device LDO:NJM2884U1 -> LDO:UT7500G-18-AB3-B-R
- U3: value UT7500G-18-AB3-B-R -> RN4020-V/RM123; device LDO:UT7500G-18-AB3-B-R -> com_module:RN4020-V/RM123
- renumbered SP2 to JP6
Connections:
- removed net INA: IC2.INA, R16.1, R17.2
- removed net INB: IC2.INB, R25.2, R26.1
- removed net N$35: C25.2, IC3.VREF, R28.2, R31.1, R32.2
- removed net N$36: C26.2, IC4.VREF, R29.2, R30.1, R33.2
- removed net N$7: R7.1, U$1.GPIO4/I2S_LROUT
- removed net N$8: R8.1, U$1.GPIO1
- removed net N$9: R9.1, U$1.GPIO0
- removed net OUTA: C17.+, IC2.OUTA, R16.2
- removed net OUTB: C18.+, IC2.OUTB, R26.2
- removed net PIO2: R3.1, U1.MLDP_EV/PIO2/CS
- removed net PIO3: R4.1, U1.WS/PIO3/MOSI
- new net FIN3: IC2.ADC7, IC6.FIN
- new net N$22: C17.1, IC3.VREF
- new net N$27: C30.1, R18.2
- new net RIN3: IC2.ADC6, IC6.RIN
- new net RST: C4.2, IC2.PC6(/RESET), J1.5, R3.2
- net +1V8: now also C10.2, IC1.CVDD0, IC1.CVDD1, IC1.CVDD2, IC1.CVDD3, U2.VOUT; no longer C14.2, U$1.CVDD0, U$1.CVDD1, U$1.CVDD2, U$1.CVDD3, U3.VOUT
- net +3V3: now also C13.1, C18.1, C5.2, C6.1, C7.2, C8.1, C9.2, IC1.AVDD0, IC1.AVDD1, IC1.AVDD2, IC1.IOVDD0, IC1.IOVDD1, IC1.IOVDD2, IC1.XTEST, IC2.AREF, IC2.AVCC, IC2.VCC@1, IC2.VCC@2, J1.2, J2.VDD, JP3.3, JP4.3, R12.1, R13.1, R3.1, R4.2, U1.VOUT, U2.VIN, U3.VDD; no longer C1.1, C12.2, C13.2, C2.1, C27.1, C4.2, IC1.AREF, IC1.AVCC, IC1.VCC@1, IC1.VCC@2, J1.VDD, JP1.3, R1.1, R14.1, R15.1, R28.1, R29.1, R34.2, U$1.AVDD0, U$1.AVDD1, U$1.AVDD2, U$1.IOVDD0, U$1.IOVDD1, U$1.IOVDD2, U$1.XTEST, U1.VDD, U2.VOUT, U3.VIN
- net BLE_RX: now also JP4.4, R8.2, U3.UART_RX; no longer IC1.PC5(ADC5/SCL), U1.UART_RX
- net BLE_TX: now also IC2.PC4(ADC4/SDA), JP4.5, U3.UART_TX; no longer IC1.PC4(ADC4/SDA), U1.UART_TX
- net CMD/MLDP: now also IC2.PD4(XCK/T0), U3.CMD/MLDP; no longer IC1.PD4(XCK/T0), U1.CMD/MLDP
- net FIN1: now also IC2.PC0(ADC0), IC4.FIN; no longer IC1.PC0(ADC0), IC3.FIN
- net FIN2: now also IC2.PC2(ADC2), IC5.FIN; no longer IC1.PC2(ADC2), IC4.FIN
- net GBUF: now also IC1.GBUF, R9.1; no longer R11.1, U$1.GBUF
- net GND: now also BAT1.-, C1.1, C10.1, C11.2, C12.2, C13.2, C15.2, C17.2, C18.2, C20.-, C21.-, C25.2, C26.2, C3.2, C5.1, C7.1, IC1.AGND0, IC1.AGND1, IC1.AGND2, IC1.AGND3, IC1.DGND0, IC1.DGND1, IC1.DGND2, IC1.DGND3, IC1.DGND4, IC1.GPIO2/DCLK, IC1.GPIO3/SDATA, IC1.GPIO6/I2S_SCLK, IC1.GPIO7/I2S_SDATA, IC2.GND@1, IC2.GND@2, IC3.!CE, IC5.GND, IC6.GND, J1.6, J2.GND, J2.SHIELD, JP3.1, JP4.1, JP5.1, R15.2, U1.GND, U3.GND@1, U3.GND@2, U3.GND@3, U3.GND@4, VR1.3; no longer C1.2, C11.1, C12.1, C13.1, C15.1, C20.1, C21.2, C25.1, C26.1, C4.1, C5.2, C7.2, IC1.GND@1, IC1.GND@2, J1.GND, J1.SHIELD, JP6.1, LED2.K, LED4.K, PWR.1, R13.2, R21.1, R24.1, R27.2, R30.2, R31.2, R8.2, R9.2, SP1.-, SP3.1, U$1.AGND0, U$1.AGND1, U$1.AGND2, U$1.AGND3, U$1.DGND0, U$1.DGND1, U$1.DGND2, U$1.DGND3, U$1.DGND4, U$1.GND, U$1.GPIO2/DCLK, U$1.GPIO3/SDATA, U$1.GPIO6/I2S_SCLK, U$1.GPIO7/I2S_SDATA, U1.GND@1, U1.GND@2, U1.GND@3, U1.GND@4, U3.GND
- net LEFT: now also IC1.LEFT, JP5.3, R11.1; no longer R19.1, R20.1, U$1.LEFT
- net MISO: now also IC1.SO, IC2.PB4(MISO), J1.1, J2.DAT0; no longer IC1.PB4(MISO), J1.DAT0, U$1.SO
- net MOSI: now also IC1.SI, IC2.PB3(MOSI/OC2), J1.4, J2.CMD; no longer IC1.PB3(MOSI/OC2), J1.CMD, U$1.SI
- net MP3-CS: now also IC1.XCS, IC2.PD6(AIN0); no longer IC1.PD6(AIN0), U$1.XCS
- net MP3-DCS: now also IC1.XDCS/BSYNC, IC2.PD7(AIN1); no longer IC1.PD7(AIN1), U$1.XDCS/BSYNC
- net MP3-DREQ: now also IC1.DREQ, IC2.PD2(INT0); no longer IC1.PD2(INT0), U$1.DREQ
- net MP3-RST: now also IC1.XRESET, IC2.PB0(ICP); no longer IC1.PB0(ICP), U$1.XRESET
- net N$1: now also IC2.PB2(SS/OC1B), LED2.A; no longer C3.2, IC1.PC6(/RESET), R1.2
- net N$10: now also C11.1, IC1.RCAP; no longer C5.1, U$1.RCAP
- net N$11: now also R15.1, U3.SPI/!PIO; no longer R13.1, U1.SPI/!PIO
- net N$12: now also IC1.RX; no longer U$1.RX
- net N$13: now also BAT1.+, JP1.2, JP2.1; no longer PWR.2, SW1.2
- net N$14: now also IC3.OUTP, JP6.1; no longer C18.-, SP1.+, SP3.2
- net N$15: now also C2.1, IC1.XTALI, R2.1; no longer C7.1, R12.1, U$1.XTALI
- net N$16: now also C14.2, R11.2; no longer C9.2, R19.2
- net N$17: now also C12.1, R9.2; no longer C6.1, R11.2
- net N$18: now also R1.2, U1.CTL; no longer R18.2, U2.CTL
- net N$19: now also C3.1, IC1.XTALO, R2.2; no longer C8.1, R12.2, U$1.XTALO
- net N$2: now also C4.1, JP3.6; no longer C3.1, JP1.6
- net N$20: now also C30.2, IC6.OUT2, JP9.1; no longer C10.1, R20.2
- net N$21: now also IC6.VREF, VR1.2; no longer C10.2, R17.1, R21.2
- net N$23: now also C16.2, IC3.AIN; no longer C15.2, R22.2
- net N$24: now also C15.1, JP5.2; no longer R23.2
- net N$25: now also C28.1, R16.2; no longer C16.2, R24.2, R25.1
- net N$26: now also C29.1, R17.2; no longer C20.2, IC2.BYPASS
- net N$29: now also IC3.OUTN; no longer C17.-
- net N$3: now also LED3.A, R14.2; no longer LED1.A, R2.2
- net N$31: now also LED1.A, R4.1; no longer LED4.A, R34.1
- net N$37: now also IC5.OUT1, JP8.2, R17.1; no longer IC4.OUT1, M2.2
- net N$38: now also C29.2, IC5.OUT2, JP8.1; no longer IC4.OUT2, M2.1
- net N$39: now also IC4.OUT1, JP7.2, R16.1; no longer IC3.OUT1, M1.2
- net N$4: now also IC2.PC5(ADC5/SCL), R8.1; no longer LED2.A, R3.2
- net N$40: now also C28.2, IC4.OUT2, JP7.1; no longer IC3.OUT2, M1.1
- net N$5: now also IC6.OUT1, JP9.2, R18.1; no longer LED3.A, R4.2
- net N$6: now also IC1.GPIO0, IC1.GPIO1, IC1.GPIO4/I2S_LROUT, IC1.GPIO5/I2S_MCLK; no longer U$1.GPIO5/I2S_MCLK
- net PIO1: now also R14.1, U3.PIO1/SCK; no longer R2.1, U1.PIO1/SCK
- net RIGHT: now also IC1.RIGHT; no longer R22.1, R23.1, U$1.RIGHT
- net RIN1: now also IC2.PC1(ADC1), IC4.RIN; no longer IC1.PC1(ADC1), IC3.RIN
- net RIN2: now also IC2.PC3(ADC3), IC5.RIN; no longer IC1.PC3(ADC3), IC4.RIN
- net RXD: now also IC2.PD0(RXD), JP3.4; no longer IC1.PD0(RXD), JP1.4
- net SCK: now also IC1.SCLK, IC2.PB5(SCK), J1.3, J2.CLK; no longer IC1.PB5(SCK), J1.CLK, U$1.SCLK
- net SD-CS: now also IC2.PB1(OC1A), J2.CD/DAT3; no longer IC1.PB1(OC1A), J1.CD/DAT3
- net SHUTDOWN: now also LED2.K, R7.1; no longer IC2.SHUTDOWN, R27.1
- net TXD: now also IC2.PD1(TXD), JP3.5; no longer IC1.PD1(TXD), JP1.5
- net VCC: now also C1.2, C20.+, C21.+, C25.1, C26.1, C27.1, IC3.VDD, IC5.VCC@1, IC5.VCC@2, IC6.VCC@1, IC6.VCC@2, JP2.2, R1.1, U1.VIN, VR1.1; no longer C11.2, C21.1, IC2.VDD, IC3.VCC@1, IC3.VCC@2, R18.1, SW1.1, U2.VIN
- net VREF1: now also IC2.PD3(INT1), IC4.VREF; no longer IC1.PD3(INT1), R32.1
- net VREF2: now also IC2.PD5(T1), IC5.VREF; no longer IC1.PD5(T1), R33.1
- net WAKE_HW: now also R12.2, U3.WAKE_HW; no longer R15.2, U1.WAKE_HW
- net WAKE_SW: now also R13.2, U3.WAKE_SW; no longer R14.2, U1.WAKE_SW
Other:
- moved on the sheet: C1, C10, C11, C12, C13, C14, C15, C16, C19, C2, C22, C23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

Commit message: 抵抗値変更
Parts:
- R16, R17, R18: value 10k -> 47
Changed lines of the file:
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@@
 <part name="C21" library="generic" deviceset="CAPACITOR-POL" device="PANASONIC_D"/>
 <part name="C28" library="generic" deviceset="CAPACITOR" device="1608_REDUCED" value="0.1u"/>
-<part name="R16" library="generic" deviceset="RESISTOR" device="1608_REDUCED" value="10k"/>
-<part name="R17" library="generic" deviceset="RESISTOR" device="1608_REDUCED" value="10k"/>
+<part name="R16" library="generic" deviceset="RESISTOR" device="1608_REDUCED" value="47"/>
+<part name="R17" library="generic" deviceset="RESISTOR" device="1608_REDUCED" value="47"/>
 <part name="C29" library="generic" deviceset="CAPACITOR" device="1608_REDUCED" value="0.1u"/>
-<part name="R18" library="generic" deviceset="RESISTOR" device="1608_REDUCED" value="10k"/>
+<part name="R18" library="generic" deviceset="RESISTOR" device="1608_REDUCED" value="47"/>
 <part name="C30" library="generic" deviceset="CAPACITOR" device="1608_REDUCED" value="0.1u"/>
 <part name="GND43" library="supply" deviceset="GND" device=""/>
