File: Development/touch_controller/touch_controller.brd (EAGLE design)
At the start: 50 x 50 mm, 44 parts, among them IC1 LPC812M101JDH16, IC2 CY8C201A0-SX2I, IC3 BMA250E, SW1 SK-12D01-VG4, U1 RN4020-V/RM123

Commit message: パラメータ決定
Parts:
- C1, C2, C3, C4, C5, C6: value (none) -> 0.1u
- R1, R12, R16, R17, R18, R19, R2: value (none) -> 10k
- R10, R11, R3, R4, R5, R6, R7, R8, R9: value (none) -> 0
- R13, R14, R15: value (none) -> 100
Changed lines of the file:
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@@
 </autorouter>
 <elements>
-<element name="C1" library="generic" package="SMD1608_REDUCED" value="" x="45.6" y="27.91" smashed="yes" rot="R90">
+<element name="C1" library="generic" package="SMD1608_REDUCED" value="0.1u" x="45.6" y="27.91" smashed="yes" rot="R90">
 <attribute name="NAME" x="47.05" y="27.41" size="0.8128" layer="25" font="vector" rot="R90"/>
 <attribute name="VALUE" x="47.25" y="27.11" size="0.8128" layer="27" font="vector" rot="R90"/>
 </element>
-<element name="C2" library="generic" package="SMD1608_REDUCED" value="" x="23.2" y="22.4" rot="R180"/>
+<element name="C2" library="generic" package="SMD1608_REDUCED" value="0.1u" x="23.2" y="22.4" rot="R180"/>
 <element name="IC1" library="micro_controller" package="TSSOP16" value="LPC812M101JDH16" x="23.56" y="17.61"/>
 <element name="SW1" library="switch" package="SK-12D01-VG4" value="SK-12D01-VG4" x="32.901709375" y="4.12385" rot="R20"/>
@@
 <attribute name="NAME" x="24.05" y="26.25" size="0.8128" layer="21" font="vector"/>
 </element>
-<element name="C3" library="generic" package="SMD1608_REDUCED" value="" x="27.4" y="28.5" smashed="yes" rot="R90">
+<element name="C3" library="generic" package="SMD1608_REDUCED" value="0.1u" x="27.4" y="28.5" smashed="yes" rot="R90">
 <attribute name="NAME" x="28.85" y="27.9" size="0.8128" layer="25" font="vector" rot="R90"/>
 <attribute name="VALUE" x="29.05" y="27.7" size="0.8128" layer="27" font="vector" rot="R90"/>
 </element>
-<element name="C4" library="generic" package="SMD1608_REDUCED" value="" x="21.5" y="28.2" smashed="yes" rot="R180">
+<element name="C4" library="generic" package="SMD1608_REDUCED" value="0.1u" x="21.5" y="28.2" smashed="yes" rot="R180">
 <attribute name="NAME" x="20.9" y="28.75" size="0.8128" layer="25" font="vector"/>
 <attribute name="VALUE" x="22.3" y="29.85" size="0.8128" layer="27" font="vector" rot="R180"/>
 </element>
-<element name="R1" library="generic" package="SMD1608_REDUCED" value="" x="22.6" y="32.8" rot="R270"/>
-<element name="R2" library="generic" package="SMD1608_REDUCED" value="" x="20.6" y="32.8" rot="R270"/>
+<element name="R1" library="generic" package="SMD1608_REDUCED" value="10k" x="22.6" y="32.8" rot="R270"/>
+<element name="R2" library="generic" package="SMD1608_REDUCED" value="10k" x="20.6" y="32.8" rot="R270"/>
 <element name="IC2" library="touch_sensor" package="SOIC-16" value="CY8C201A0-SX2I" x="13.5" y="25" smashed="yes" rot="R180">
 <attribute name="NAME" x="8.2" y="24.3" size="0.8128" layer="25" font="vector" rot="SR90"/>
 </element>
-<element name="C5" library="generic" package="SMD1608_REDUCED" value="" x="17.9" y="19.6" rot="R270"/>
-<element name="C6" library="generic" package="SMD1608_REDUCED" value="" x="16.7" y="30.5" rot="R270"/>
-<element name="R3" library="generic" package="SMD1608_REDUCED" value="" x="25" y="45.1" rot="R90"/>
-<element name="R4" library="generic" package="SMD1608_REDUCED" value="" x="38.2" y="41.3"/>
-<element name="R5" library="generic" package="SMD1608_REDUCED" value="" x="48" y="21.5" rot="R90"/>
-<element name="R6" library="generic" package="SMD1608_REDUCED" value="" x="38.3" y="8.7" smashed="yes">
+<element name="C5" library="generic" package="SMD1608_REDUCED" value="0.1u" x="17.9" y="19.6" rot="R270"/>
+<element name="C6" library="generic" package="SMD1608_REDUCED" value="0.1u" x="16.7" y="30.5" rot="R270"/>
+<element name="R3" library="generic" package="SMD1608_REDUCED" value="0" x="25" y="45.1" rot="R90"/>
+<element name="R4" library="generic" package="SMD1608_REDUCED" value="0" x="38.2" y="41.3"/>
+<element name="R5" library="generic" package="SMD1608_REDUCED" value="0" x="48" y="21.5" rot="R90"/>
+<element name="R6" library="generic" package="SMD1608_REDUCED" value="0" x="38.3" y="8.7" smashed="yes">
 <attribute name="NAME" x="37.6" y="7.25" size="0.8128" layer="25" font="vector"/>
 <attribute name="VALUE" x="37.5" y="7.05" size="0.8128" layer="27" font="vector"/>
 </element>
-<element name="R7" library="generic" package="SMD1608_REDUCED" value="" x="24.1" y="5.7"/>
-<element name="R8" library="generic" package="SMD1608_REDUCED" value="" x="8.8" y="11.7" rot="R270"/>
-<element name="R9" library="generic" package="SMD1608_REDUCED" value="" x="4.9" y="25" rot="R180"/>
-<element name="R10" library="generic" package="SMD1608_REDUCED" value="" x="8.8" y="37.5" rot="R90"/>
-<element name="R11" library="generic" package="SMD1608_REDUCED" value="" x="21.5" y="25.6" smashed="yes">
+<element name="R7" library="generic" package="SMD1608_REDUCED" value="0" x="24.1" y="5.7"/>
+<element name="R8" library="generic" package="SMD1608_REDUCED" value="0" x="8.8" y="11.7" rot="R270"/>
+<element name="R9" library="generic" package="SMD1608_REDUCED" value="0" x="4.9" y="25" rot="R180"/>
+<element name="R10" library="generic" package="SMD1608_REDUCED" value="0" x="8.8" y="37.5" rot="R90"/>
+<element name="R11" library="generic" package="SMD1608_REDUCED" value="0" x="21.5" y="25.6" smashed="yes">
 <attribute name="NAME" x="20.5" y="24.15" size="0.8128" layer="25" font="vector"/>
 <attribute name="VALUE" x="20.7" y="23.95" size="0.8128" layer="27" font="vector"/>
 </element>
-<element name="R12" library="generic" package="SMD1608_REDUCED" value="" x="23.5" y="13" rot="R180"/>
+<element name="R12" library="generic" package="SMD1608_REDUCED" value="10k" x="23.5" y="13" rot="R180"/>
 <element name="LED1" library="generic" package="LED1608_REDUCED" value="" x="31" y="16.2" smashed="yes" rot="R180">
 <attribute name="NAME" x="26.7" y="15.85" size="0.8128" layer="25" font="vector"/>
@@
 <attribute name="VALUE" x="31.8" y="14.95" size="0.8128" layer="27" font="vector" rot="R180"/>
 </element>
-<element name="R13" library="generic" package="SMD1608_REDUCED" value="" x="34.4" y="16.2" smashed="yes" rot="R180">
+<element name="R13" library="generic" package="SMD1608_REDUCED" value="100" x="34.4" y="16.2" smashed="yes" rot="R180">
 <attribute name="NAME" x="36" y="15.85" size="0.8128" layer="25" font="vector"/>
 <attribute name="VALUE" x="35.2" y="17.85" size="0.8128" layer="27" font="vector" rot="R180"/>
 </element>
-<element name="R14" library="generic" package="SMD1608_REDUCED" value="" x="34.4" y="14.8" smashed="yes" rot="R180">
+<element name="R14" library="generic" package="SMD1608_REDUCED" value="100" x="34.4" y="14.8" smashed="yes" rot="R180">
 <attribute name="NAME" x="36" y="14.45" size="0.8128" layer="25" font="vector"/>
 <attribute name="VALUE" x="35.2" y="16.45" size="0.8128" layer="27" font="vector" rot="R180"/>
 </element>
-<element name="R15" library="generic" package="SMD1608_REDUCED" value="" x="34.4" y="13.3" smashed="yes" rot="R180">
+<element name="R15" library="generic" package="SMD1608_REDUCED" value="100" x="34.4" y="13.3" smashed="yes" rot="R180">
 <attribute name="NAME" x="36" y="12.95" size="0.8128" layer="25" font="vector"/>
 <attribute name="VALUE" x="35.2" y="14.95" size="0.8128" layer="27" font="vector" rot="R180"/>
 </element>
-<element name="R16" library="generic" package="SMD1608_REDUCED" value="" x="30.9" y="19.1" smashed="yes" rot="R270">
+<element name="R16" library="generic" package="SMD1608_REDUCED" value="10k" x="30.9" y="19.1" smashed="yes" rot="R270">
 <attribute name="NAME" x="30.35" y="18.2" size="0.8128" layer="25" font="vector" rot="R90"/>
 <attribute name="VALUE" x="29.25" y="19.9" size="0.8128" layer="27" font="vector" rot="R270"/>
 </element>
-<element name="R17" library="generic" package="SMD1608_REDUCED" value="" x="30.9" y="22.4" smashed="yes" rot="R270">
+<element name="R17" library="generic" package="SMD1608_REDUCED" value="10k" x="30.9" y="22.4" smashed="yes" rot="R270">
 <attribute name="NAME" x="30.25" y="21.5" size="0.8128" layer="25" font="vector" rot="R90"/>
 <attribute name="VALUE" x="29.25" y="23.2" size="0.8128" layer="27" font="vector" rot="R270"/>
 </element>
-<element name="R18" library="generic" package="SMD1608_REDUCED" value="" x="41.3" y="15.3" rot="R90"/>
-<element name="R19" library="generic" package="SMD1608_REDUCED" value="" x="45.5" y="21.3" smashed="yes" rot="R90">
+<element name="R18" library="generic" package="SMD1608_REDUCED" value="10k" x="41.3" y="15.3" rot="R90"/>
+<element name="R19" library="generic" package="SMD1608_REDUCED" value="10k" x="45.5" y="21.3" smashed="yes" rot="R90">
 <attribute name="NAME" x="45.95" y="17.7" size="0.8128" layer="25" font="vector" rot="R90"/>
 <attribute name="VALUE" x="47.15" y="20.5" size="0.8128" layer="27" font="vector" rot="R90"/>

Commit message: touch_controller rev2
Parts:
- added C7, C8: 0.1u, generic:SMD1608_REDUCED
- added LED4: (no value), generic:LED1608_REDUCED
- added R20: 1k, generic:SMD1608_REDUCED
- added U$1: M03X2STD, header:2X03
- IC1: value LPC812M101JDH16 -> ATMEGA328P-AU; device micro_controller:TSSOP16 -> AVR:TQFP32-08
- moved R4 14.4 mm to (23.8, 42.0), turned to 270 degrees
- moved IC1 14.4 mm to (11.6, 25.6)
- moved C5 14.2 mm to (21.5, 33.3), turned to 0 degrees
- moved IC2 13.0 mm to (16.2, 37.7)
- moved C6 12.0 mm to (20.3, 41.9), turned to 180 degrees
- moved C2 8.73 mm to (20.5, 14.1), turned to 90 degrees
- moved C3 8.40 mm to (27.5, 20.1)
- moved IC3 8.40 mm to (25.0, 20.1)
- moved R1 8.22 mm to (22.0, 24.6)
- moved R2 8.20 mm to (20.5, 24.6)
- moved C4 7.44 mm to (22.3, 20.8), turned to 90 degrees
- moved R5 6.20 mm to (48.0, 27.7), turned to 270 degrees
- moved R6 4.17 mm to (41.3, 11.6), turned to 270 degrees
- moved R9 3.50 mm to (3.10, 28.0), turned to 270 degrees
- moved R11 2.97 mm to (24.0, 27.2)
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Connections:
- removed net ISP_EN: IC1.2, JP1.6
- removed net ISP_RXD: IC1.16, JP1.4
- removed net ISP_TXD: IC1.4, JP1.5
- new net MISO: IC1.16, U$1.1
- new net MOSI: IC1.15, U$1.4
- new net N$13: IC1.11, R20.2
- new net N$17: LED4.A, R20.1
- new net RESET: C2.1, JP1.6
- new net RXD: IC1.30, JP1.4
- new net SCK: IC1.17, U$1.3
- new net TXD: IC1.31, JP1.5
- net +3V3: now also C7.2, C8.2, IC1.18, IC1.20, IC1.4, IC1.6, U$1.2; no longer C2.1, IC1.12
- net BLE_RX: now also IC1.32; no longer IC1.14
- net BLE_TX: now also IC1.1; no longer IC1.15
- net GND: now also C7.1, C8.1, IC1.21, IC1.3, IC1.5, LED4.K, U$1.6; no longer C2.2, IC1.13
- net RST: now also C2.2, IC1.29, U$1.5; no longer IC1.3, JP1.2
- net SCL: now also IC1.28; no longer IC1.7
- net SDA: now also IC1.27; no longer IC1.8
- net WAKE_HW: now also IC1.2; no longer IC1.11
Routing:
- net +3V3: track 124.3 -> 165.1 mm, vias 0 -> 1
- net GND: track 152.5 -> 118.9 mm, vias 60 -> 91
- net GP0_4: track 30.3 -> 60.5 mm, vias 0 -> 2
- net TXD: track 0.00 -> 28.5 mm, vias 0 -> 1
- net RXD: track 0.00 -> 28.4 mm, vias 0 -> 1
- net GP0_1: track 34.6 -> 11.4 mm
- net WAKE_HW: track 20.7 -> 42.7 mm, vias 0 -> 2
- net WAKE_SW: track 7.54 -> 27.3 mm, vias 0 -> 2
- net GP0_0: track 28.8 -> 9.09 mm
- net ISP_RXD: track 19.3 -> 0.00 mm
- net CMD/MLDP: track 8.81 -> 26.7 mm, vias 0 -> 2
- net GP0_2: track 51.3 -> 34.7 mm
- net GP1_0: track 25.5 -> 42.1 mm
- net N$4: track 2.20 -> 17.6 mm
- net BLE_TX: track 18.0 -> 32.4 mm
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Other:
- outline, holes or cut-outs redrawn
- board text added: "KENBISHI TOUCH CONTROLLER"
- board text added: "Rev.2"
- board text removed: "KENBISHI"
- board text removed: "Rev 1"
- board text removed: "Touch Controller"

Commit message: rev3設計完了
Parts:
- removed R12, R16, R17, R18, R19: 10k, generic:SMD1608_REDUCED
- removed R13, R14, R15: 100, generic:SMD1608_REDUCED
- removed R20: 1k, generic:SMD1608_REDUCED
- removed TP4, TP5, TP6, TP7, TP8, TP9: HT-0720-10, test_pin:HT-0720-10
- added C10, C9: 0.1u, generic:SMD1608_REDUCED
- added IC4: CY8C201A0-SX2I, touch_sensor:SOIC-16
- C1, C2: value 0.1u -> 10u; device generic:SMD1608_REDUCED -> generic:SMD2012_REDUCED
- IC1: value ATMEGA328P-AU -> XCL101; device AVR:TQFP32-08 -> DCDC:CL-2025
- IC2: value CY8C201A0-SX2I -> ATMEGA328P-AU; device touch_sensor:SOIC-16 -> AVR:TQFP32-08
- R10, R11, R9: value 0 -> 100
- R2: value 10k -> 1k
- R3, R4, R5, R6, R7, R8: value 0 -> 10k
- moved R8 37.9 mm to (45.5, 21.3), turned to 90 degrees
- moved TP3 34.9 mm to (19.4, 45.0)
- moved R10 34.2 mm to (34.4, 14.8), turned to 180 degrees
- moved R9 33.5 mm to (34.4, 16.2), turned to 180 degrees
- moved LED4 29.1 mm to (31.0, 13.3), turned to 180 degrees
- moved C1 28.9 mm to (26.6, 6.10)
- moved LED1 28.6 mm to (2.70, 20.1), turned to 90 degrees
- moved TP2 27.4 mm to (14.2, 45.0)
- moved IC1 23.6 mm to (23.2, 5.10), turned to 90 degrees
- moved C6 23.0 mm to (27.5, 20.1), turned to 90 degrees
- moved R3 20.6 mm to (22.0, 24.6), turned to 270 degrees
- moved R4 17.7 mm to (20.5, 24.6)
- moved R11 17.4 mm to (34.4, 13.3), turned to 180 degrees
- moved C4 17.3 mm to (5.40, 24.7), turned to 270 degrees
- moved C7 17.3 mm to (22.3, 20.8), turned to 90 degrees
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Connections:
- removed net N$10: R10.2, TP8.P$1
- removed net N$11: R11.2, TP9.P$1
- removed net N$3: R3.2, TP1.P$1
- removed net N$4: R4.2, TP2.P$1
- removed net N$5: R5.2, TP3.P$1
- removed net N$6: R6.2, TP4.P$1
- removed net N$7: R7.2, TP5.P$1
- removed net N$8: R8.2, TP6.P$1
- removed net N$9: R9.2, TP7.P$1
- new net N$18: C2.1, IC1.3, IC1.4, IC1.8, SW1.3
- new net N$20: IC1.1, IC1.7
- net +3V3: now also C10.1, C4.2, C5.2, C6.1, C7.1, C9.1, IC1.2, IC2.18, IC2.20, IC2.4, IC2.6, IC4.16, R3.1, R4.1, R5.1, R6.1; no longer C3.1, C4.1, C5.1, C7.2, C8.2, IC1.18, IC1.20, IC1.4, IC1.6, IC2.16, R12.1, R17.1, R18.1, R2.1, SW1.3
- net BLE_RX: now also IC2.32; no longer IC1.32
- net BLE_TX: now also IC2.1; no longer IC1.1
- net CMD/MLDP: now also IC2.10, R7.1; no longer IC1.10, R16.1
- net GND: now also C10.2, C2.2, C4.1, C5.1, C6.2, C7.2, C9.2, IC1.6, IC2.21, IC2.3, IC2.5, IC4.10, R7.2, R8.2; no longer C3.2, C4.2, C5.2, C6.1, C7.1, IC1.21, IC1.3, IC1.5, IC2.10, R16.2, R19.2
- net GP0_0: now also IC4.4, TP1.P$1; no longer IC2.4, R3.1
- net GP0_1: now also IC4.5, TP2.P$1; no longer IC2.5, R4.1
- net GP0_2: now also IC4.15, TP3.P$1; no longer IC2.15, R5.1
- net GP0_3: now also IC4.1; no longer IC2.1, R6.1
- net GP0_4: now also IC4.3; no longer IC2.3, R7.1
- net GP1_0: now also IC4.8; no longer IC2.8, R8.1
- net GP1_1: now also IC4.9; no longer IC2.9, R9.1
- net GP1_2: now also IC4.11; no longer IC2.11, R10.1
- net GP1_3: now also IC4.12; no longer IC2.12, R11.1
- net GP1_4: now also IC4.13; no longer IC2.13
- net MISO: now also IC2.16; no longer IC1.16
- net MOSI: now also IC2.15; no longer IC1.15
- net N$12: now also R8.1; no longer R19.1
- net N$13: now also IC2.11, R2.2; no longer IC1.11, R20.2
- net N$14: now also LED2.A, R9.2; no longer LED1.A, R13.2
- net N$15: now also LED3.A, R10.2; no longer LED2.A, R14.2
- net N$16: now also LED4.A, R11.2; no longer LED3.A, R15.2
- net N$17: now also LED1.A, R2.1; no longer LED4.A, R20.1
- net N$2: now also C8.2, IC4.2; no longer C6.2, IC2.2
- net PIO1: now also R9.1; no longer R13.1
- net PIO2: now also R10.1; no longer R14.1
- net PIO3: now also R11.1; no longer R15.1
- net RESET: now also C3.1; no longer C2.1
- net RST: now also C3.2, IC2.29, R1.2; no longer C2.2, IC1.29, R12.2
- net RXD: now also IC2.30; no longer IC1.30
- net SCK: now also IC2.17; no longer IC1.17
- net SCL: now also IC2.28, IC4.6, R3.2; no longer IC1.28, IC2.6, R1.2
- net SDA: now also IC2.27, IC4.7, R4.2; no longer IC1.27, IC2.7, R2.2
- net TXD: now also IC2.31; no longer IC1.31
- net WAKE_HW: now also IC2.2, R5.2; no longer IC1.2, R18.2
- net WAKE_SW: now also IC2.9, R6.2; no longer IC1.9, R17.2
Routing:
- net GP0_4: track 60.5 -> 0.00 mm, vias 2 -> 0
- net GP0_3: track 56.4 -> 0.00 mm
- net GP1_0: track 42.1 -> 0.00 mm
- net GP0_2: track 34.7 -> 11.7 mm
- net N$18: track 0.00 -> 19.2 mm, vias 0 -> 1
- net N$4: track 17.6 -> 0.00 mm
- net GP1_2: track 16.4 -> 0.00 mm
- net GP1_1: track 12.7 -> 0.00 mm
- net GP1_3: track 12.5 -> 0.00 mm
- net GP0_1: track 11.4 -> 4.97 mm
- net GP0_0: track 9.09 -> 4.44 mm
- net N$7: track 3.71 -> 0.00 mm
- net N$10: track 2.98 -> 0.00 mm
- net N$20: track 0.00 -> 2.61 mm
- net N$9: track 2.58 -> 0.00 mm
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Other:
- board text added: "Rev.3"
- board text removed: "Rev.2"
