File: Development/touch_controller/touch_controller.sch (EAGLE design)
At the start: 44 parts, among them IC1 LPC812M101JDH16, IC2 CY8C201A0-SX2I, IC3 BMA250E, SW1 SK-12D01-VG4, U1 RN4020-V/RM123

Commit message: パラメータ決定
Parts:
- C1, C2, C3, C4, C5, C6: value (none) -> 0.1u
- R1, R12, R16, R17, R18, R19, R2: value (none) -> 10k
- R10, R11, R3, R4, R5, R6, R7, R8, R9: value (none) -> 0
- R13, R14, R15: value (none) -> 100
Changed lines of the file:
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@@
 <part name="U1" library="com_module" deviceset="RN4020" device="-V/RM123"/>
 <part name="IC1" library="micro_controller" deviceset="LPC812M101JDH16" device=""/>
-<part name="C1" library="generic" deviceset="CAPACITOR" device="1608_REDUCED"/>
-<part name="C2" library="generic" deviceset="CAPACITOR" device="1608_REDUCED"/>
+<part name="C1" library="generic" deviceset="CAPACITOR" device="1608_REDUCED" value="0.1u"/>
+<part name="C2" library="generic" deviceset="CAPACITOR" device="1608_REDUCED" value="0.1u"/>
 <part name="+3V1" library="supply" deviceset="+3V3" device=""/>
 <part name="+3V2" library="supply" deviceset="+3V3" device=""/>
@@
 <part name="+3V4" library="supply" deviceset="+3V3" device=""/>
 <part name="GND9" library="supply" deviceset="GND" device=""/>
-<part name="C3" library="generic" deviceset="CAPACITOR" device="1608_REDUCED"/>
-<part name="C4" library="generic" deviceset="CAPACITOR" device="1608_REDUCED"/>
+<part name="C3" library="generic" deviceset="CAPACITOR" device="1608_REDUCED" value="0.1u"/>
+<part name="C4" library="generic" deviceset="CAPACITOR" device="1608_REDUCED" value="0.1u"/>
 <part name="+3V5" library="supply" deviceset="+3V3" device=""/>
 <part name="GND10" library="supply" deviceset="GND" device=""/>
@@
 <part name="+3V6" library="supply" deviceset="+3V3" device=""/>
 <part name="GND13" library="supply" deviceset="GND" device=""/>
-<part name="R1" library="generic" deviceset="RESISTOR" device="1608_REDUCED"/>
-<part name="R2" library="generic" deviceset="RESISTOR" device="1608_REDUCED"/>
+<part name="R1" library="generic" deviceset="RESISTOR" device="1608_REDUCED" value="10k"/>
+<part name="R2" library="generic" deviceset="RESISTOR" device="1608_REDUCED" value="10k"/>
 <part name="+3V7" library="supply" deviceset="+3V3" device=""/>
 <part name="+3V8" library="supply" deviceset="+3V3" device=""/>
@@
 <part name="+3V9" library="supply" deviceset="+3V3" device=""/>
 <part name="GND15" library="supply" deviceset="GND" device=""/>
-<part name="C5" library="generic" deviceset="CAPACITOR" device="1608_REDUCED"/>
-<part name="C6" library="generic" deviceset="CAPACITOR" device="1608_REDUCED"/>
+<part name="C5" library="generic" deviceset="CAPACITOR" device="1608_REDUCED" value="0.1u"/>
+<part name="C6" library="generic" deviceset="CAPACITOR" device="1608_REDUCED" value="0.1u"/>
 <part name="GND16" library="supply" deviceset="GND" device=""/>
-<part name="R3" library="generic" deviceset="RESISTOR" device="1608_REDUCED"/>
-<part name="R4" library="generic" deviceset="RESISTOR" device="1608_REDUCED"/>
-<part name="R5" library="generic" deviceset="RESISTOR" device="1608_REDUCED"/>
-<part name="R6" library="generic" deviceset="RESISTOR" device="1608_REDUCED"/>
-<part name="R7" library="generic" deviceset="RESISTOR" device="1608_REDUCED"/>
-<part name="R8" library="generic" deviceset="RESISTOR" device="1608_REDUCED"/>
-<part name="R9" library="generic" deviceset="RESISTOR" device="1608_REDUCED"/>
-<part name="R10" library="generic" deviceset="RESISTOR" device="1608_REDUCED"/>
-<part name="R11" library="generic" deviceset="RESISTOR" device="1608_REDUCED"/>
-<part name="R12" library="generic" deviceset="RESISTOR" device="1608_REDUCED"/>
+<part name="R3" library="generic" deviceset="RESISTOR" device="1608_REDUCED" value="0"/>
+<part name="R4" library="generic" deviceset="RESISTOR" device="1608_REDUCED" value="0"/>
+<part name="R5" library="generic" deviceset="RESISTOR" device="1608_REDUCED" value="0"/>
+<part name="R6" library="generic" deviceset="RESISTOR" device="1608_REDUCED" value="0"/>
+<part name="R7" library="generic" deviceset="RESISTOR" device="1608_REDUCED" value="0"/>
+<part name="R8" library="generic" deviceset="RESISTOR" device="1608_REDUCED" value="0"/>
+<part name="R9" library="generic" deviceset="RESISTOR" device="1608_REDUCED" value="0"/>
+<part name="R10" library="generic" deviceset="RESISTOR" device="1608_REDUCED" value="0"/>
+<part name="R11" library="generic" deviceset="RESISTOR" device="1608_REDUCED" value="0"/>
+<part name="R12" library="generic" deviceset="RESISTOR" device="1608_REDUCED" value="10k"/>
 <part name="+3V10" library="supply" deviceset="+3V3" device=""/>
 <part name="LED1" library="generic" deviceset="LED" device="1608_REDUCED"/>
@@
 <part name="GND18" library="supply" deviceset="GND" device=""/>
 <part name="GND19" library="supply" deviceset="GND" device=""/>
-<part name="R13" library="generic" deviceset="RESISTOR" device="1608_REDUCED"/>
-<part name="R14" library="generic" deviceset="RESISTOR" device="1608_REDUCED"/>
-<part name="R15" library="generic" deviceset="RESISTOR" device="1608_REDUCED"/>
-<part name="R16" library="generic" deviceset="RESISTOR" device="1608_REDUCED"/>
-<part name="R17" library="generic" deviceset="RESISTOR" device="1608_REDUCED"/>
+<part name="R13" library="generic" deviceset="RESISTOR" device="1608_REDUCED" value="100"/>
+<part name="R14" library="generic" deviceset="RESISTOR" device="1608_REDUCED" value="100"/>
+<part name="R15" library="generic" deviceset="RESISTOR" device="1608_REDUCED" value="100"/>
+<part name="R16" library="generic" deviceset="RESISTOR" device="1608_REDUCED" value="10k"/>
+<part name="R17" library="generic" deviceset="RESISTOR" device="1608_REDUCED" value="10k"/>
 <part name="+3V11" library="supply" deviceset="+3V3" device=""/>
 <part name="GND20" library="supply" deviceset="GND" device=""/>
-<part name="R18" library="generic" deviceset="RESISTOR" device="1608_REDUCED"/>
-<part name="R19" library="generic" deviceset="RESISTOR" device="1608_REDUCED"/>
+<part name="R18" library="generic" deviceset="RESISTOR" device="1608_REDUCED" value="10k"/>
+<part name="R19" library="generic" deviceset="RESISTOR" device="1608_REDUCED" value="10k"/>
 <part name="GND21" library="supply" deviceset="GND" device=""/>
 <part name="GND22" library="supply" deviceset="GND" device=""/>

Commit message: touch_controller rev2
Parts:
- added C7, C8: 0.1u, generic:CAPACITOR1608_REDUCED
- added LED4: (no value), generic:LED1608_REDUCED
- added R20: 1k, generic:RESISTOR1608_REDUCED
- added U$1: M03X2STD, header:M03X2STD
- IC1: value LPC812M101JDH16 -> ATMEGA328P-AU; device micro_controller:LPC812M101JDH16 -> AVR:ATMEGA328P-AU
Connections:
- removed net ISP_EN: IC1.PIO0_12, JP1.6
- removed net ISP_RXD: IC1.PIO0_0/ACMP_I1/TDO, JP1.4
- removed net ISP_TXD: IC1.PIO0_4/WAKEUP/!TRST, JP1.5
- new net MISO: IC1.PB4(MISO), U$1.1
- new net MOSI: IC1.PB3(MOSI/OC2), U$1.4
- new net N$13: IC1.PD7(AIN1), R20.2
- new net N$17: LED4.A, R20.1
- new net RESET: C2.1, JP1.6
- new net RXD: IC1.PD0(RXD), JP1.4
- new net SCK: IC1.PB5(SCK), U$1.3
- new net TXD: IC1.PD1(TXD), JP1.5
- net +3V3: now also C7.2, C8.2, IC1.AREF, IC1.AVCC, IC1.VCC@1, IC1.VCC@2, U$1.2; no longer C2.1, IC1.VDD
- net BLE_RX: now also IC1.PD2(INT0); no longer IC1.PIO0_7
- net BLE_TX: now also IC1.PD3(INT1); no longer IC1.PIO0_6/VDDCMP
- net CMD/MLDP: now also IC1.PD6(AIN0); no longer IC1.PIO0_9/XTALOUT
- net GND: now also C7.1, C8.1, IC1.GND, IC1.GND@1, IC1.GND@2, LED4.K, U$1.6; no longer C2.2, IC1.VSS
- net RST: now also C2.2, IC1.PC6(/RESET), U$1.5; no longer IC1.!RESET!/PIO0_5, JP1.2
- net SCL: now also IC1.PC5(ADC5/SCL); no longer IC1.PIO0_11
- net SDA: now also IC1.PC4(ADC4/SDA); no longer IC1.PIO0_10
- net WAKE_HW: now also IC1.PD4(XCK/T0); no longer IC1.PIO0_8/XTALIN
- net WAKE_SW: now also IC1.PD5(T1); no longer IC1.PIO0_1/ACMP_I2/CLKIN/TDI
Other:
- moved on the sheet: C2, R12

Commit message: rev3設計完了
Parts:
- removed R12, R16, R17, R18, R19: 10k, generic:RESISTOR1608_REDUCED
- removed R13, R14, R15: 100, generic:RESISTOR1608_REDUCED
- removed R20: 1k, generic:RESISTOR1608_REDUCED
- removed TP4, TP5, TP6, TP7, TP8, TP9: HT-0720-10, test_pin:HT-0720-10
- added C10, C9: 0.1u, generic:CAPACITOR1608_REDUCED
- added IC4: CY8C201A0-SX2I, touch_sensor:CY8C201A0-SX2I
- C1, C2: value 0.1u -> 10u; device generic:CAPACITOR1608_REDUCED -> generic:CAPACITOR2012_REDUCED
- IC1: value ATMEGA328P-AU -> XCL101; device AVR:ATMEGA328P-AU -> DCDC:XCL101
- IC2: value CY8C201A0-SX2I -> ATMEGA328P-AU; device touch_sensor:CY8C201A0-SX2I -> AVR:ATMEGA328P-AU
- R10, R11, R9: value 0 -> 100
- R2: value 10k -> 1k
- R3, R4, R5, R6, R7, R8: value 0 -> 10k
Connections:
- removed net N$10: R10.2, TP8.P$1
- removed net N$11: R11.2, TP9.P$1
- removed net N$3: R3.2, TP1.P$1
- removed net N$4: R4.2, TP2.P$1
- removed net N$5: R5.2, TP3.P$1
- removed net N$6: R6.2, TP4.P$1
- removed net N$7: R7.2, TP5.P$1
- removed net N$8: R8.2, TP6.P$1
- removed net N$9: R9.2, TP7.P$1
- new net N$18: C2.1, IC1.CE, IC1.L2, IC1.VBAT, SW1.P$3
- new net N$20: IC1.L1, IC1.LX
- net +3V3: now also C10.1, C4.2, C5.2, C6.1, C7.1, C9.1, IC1.VOUT, IC2.AREF, IC2.AVCC, IC2.VCC@1, IC2.VCC@2, IC4.VDD, R3.1, R4.1, R5.1, R6.1; no longer C3.1, C4.1, C5.1, C7.2, C8.2, IC1.AREF, IC1.AVCC, IC1.VCC@1, IC1.VCC@2, IC2.VDD, R12.1, R17.1, R18.1, R2.1, SW1.P$3
- net BLE_RX: now also IC2.PD2(INT0); no longer IC1.PD2(INT0)
- net BLE_TX: now also IC2.PD3(INT1); no longer IC1.PD3(INT1)
- net CMD/MLDP: now also IC2.PD6(AIN0), R7.1; no longer IC1.PD6(AIN0), R16.1
- net GND: now also C10.2, C2.2, C4.1, C5.1, C6.2, C7.2, C9.2, IC1.VSS, IC2.GND, IC2.GND@1, IC2.GND@2, IC4.VSS, R7.2, R8.2; no longer C3.2, C4.2, C5.2, C6.1, C7.1, IC1.GND, IC1.GND@1, IC1.GND@2, IC2.VSS, R16.2, R19.2
- net GP0_0: now also IC4.GP0_0, TP1.P$1; no longer IC2.GP0_0, R3.1
- net GP0_1: now also IC4.GP0_1, TP2.P$1; no longer IC2.GP0_1, R4.1
- net GP0_2: now also IC4.GP0_2, TP3.P$1; no longer IC2.GP0_2, R5.1
- net GP0_3: now also IC4.GP0_3; no longer IC2.GP0_3, R6.1
- net GP0_4: now also IC4.GP0_4; no longer IC2.GP0_4, R7.1
- net GP1_0: now also IC4.GP1_0; no longer IC2.GP1_0, R8.1
- net GP1_1: now also IC4.GP1_1; no longer IC2.GP1_1, R9.1
- net GP1_2: now also IC4.GP1_2; no longer IC2.GP1_2, R10.1
- net GP1_3: now also IC4.GP1_3; no longer IC2.GP1_3, R11.1
- net GP1_4: now also IC4.GP1_4; no longer IC2.GP1_4
- net MISO: now also IC2.PB4(MISO); no longer IC1.PB4(MISO)
- net MOSI: now also IC2.PB3(MOSI/OC2); no longer IC1.PB3(MOSI/OC2)
- net N$12: now also R8.1; no longer R19.1
- net N$13: now also IC2.PD7(AIN1), R2.2; no longer IC1.PD7(AIN1), R20.2
- net N$14: now also LED2.A, R9.2; no longer LED1.A, R13.2
- net N$15: now also LED3.A, R10.2; no longer LED2.A, R14.2
- net N$16: now also LED4.A, R11.2; no longer LED3.A, R15.2
- net N$17: now also LED1.A, R2.1; no longer LED4.A, R20.1
- net N$2: now also C8.2, IC4.CSINT; no longer C6.2, IC2.CSINT
- net PIO1: now also R9.1; no longer R13.1
- net PIO2: now also R10.1; no longer R14.1
- net PIO3: now also R11.1; no longer R15.1
- net RESET: now also C3.1; no longer C2.1
- net RST: now also C3.2, IC2.PC6(/RESET), R1.2; no longer C2.2, IC1.PC6(/RESET), R12.2
- net RXD: now also IC2.PD0(RXD); no longer IC1.PD0(RXD)
- net SCK: now also IC2.PB5(SCK); no longer IC1.PB5(SCK)
- net SCL: now also IC2.PC5(ADC5/SCL), IC4.I2CSCL, R3.2; no longer IC1.PC5(ADC5/SCL), IC2.I2CSCL, R1.2
- net SDA: now also IC2.PC4(ADC4/SDA), IC4.I2CSDA, R4.2; no longer IC1.PC4(ADC4/SDA), IC2.I2CSDA, R2.2
- net TXD: now also IC2.PD1(TXD); no longer IC1.PD1(TXD)
- net WAKE_HW: now also IC2.PD4(XCK/T0), R5.2; no longer IC1.PD4(XCK/T0), R18.2
- net WAKE_SW: now also IC2.PD5(T1), R6.2; no longer IC1.PD5(T1), R17.2
Other:
- moved on the sheet: BAT1, C1, C2, C3, C4, C5, C6, C7, C8, LED1, LED2, LED3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
